Commit message: removing virtual mode

File: urdf/pioneer3dx.xacro (robot description, xacro)
@@ -25,7 +25,7 @@
 		<origin xyz=".18 0 0.025" rpy="0 0 0"/>
 		<parent link="top_plate"/>
-		<child link="base_laser"/>
-	</joint>
-	<link name="base_laser">
+		<child link="laser"/>
+	</joint>
+	<link name="laser">
 		<collision>
 			<origin xyz="0 0 0" rpy="0 0 0"/>
