Commit message: completed urdf

File: p2os_description/urdf/pioneer3dx/pioneer3dx.xacro (robot description, xacro)
@@ -5,5 +5,5 @@
 	xmlns:interface="http://playerstage.sourceforge.net/gazebo/xmlschema/#interface"
 	xmlns:xacro="http://ros.org/wiki/xacro">
-  <include filename="$(find p2os_urdf)/defs/pioneer3dx_wheel.xacro"/>
+  <xacro:include filename="$(find p2os_urdf)/defs/pioneer3dx_wheel.xacro"/>
 <!-- Chassis -->
 	<link name="base_link">
@@ -21,29 +21,4 @@
 		<material value="Gazebo/Red"/>
 	</gazebo>
-<!-- Laser -->
-	<joint name="hokuyo_joint" type="fixed">
-		<origin xyz=".18 0 0.025" rpy="0 0 0"/>
-		<parent link="top_plate"/>
-		<child link="laser"/>
-	</joint>
-	<link name="laser">
-		<collision>
-			<origin xyz="0 0 0" rpy="0 0 0"/>
-				<geometry>
-					<box size="0.05 0.05 0.05"/>
-				</geometry>
-		</collision>
-		<visual>
-			<origin xyz="0 0 0" rpy="0 0 0"/>
-			<geometry>
-				<box size="0.05 0.05 0.05"/>
-			</geometry>
-		</visual>
-		<inertial>
-			<mass value="1e-5" />
-			<origin xyz="0 0 0" rpy="0 0 0"/>
-			<inertia ixx="1e-6" ixy="0" ixz="0" iyy="1e-6" iyz="0" izz="1e-6" />
-		</inertial>
-	</link>
 <!-- Top -->
 	<joint name="base_top_joint" type="fixed">
